File: Buck Boost.kicad_pcb (KiCad board)
At the start: 2 copper layers, 36 parts, among them J1 Screw_Terminal_01x02, J3 Screw_Terminal_01x02, K2 Jumper_2_Bridged, T2 IRF4905, T3 IRF4905, U1 HCPL-3120, U2 arduino, U3 HCPL-3120, U4 ER_OLEDM0.91_1x-I2C, U5 TMA-1512S

Commit message: smd
Parts:
- removed LED3: CQY99, LED_THT:LED_D5.0mm_IRGrey
- removed R5: R, Resistor_THT:R_Axial_DIN0204_L3.6mm_D1.6mm_P7.62mm_Horizontal
- added C9: 1uF, Capacitor_SMD:C_0805_2012Metric, F.Cu at (190.8, 105.1)
- added J2: DC 5V, TerminalBlock_MetzConnect:TerminalBlock_MetzConnect_360381_1x01_Horizontal_ScrewM3.0, F.Cu at (119.4, 122.2)
- added J4: TRACO DC IN, TerminalBlock_MetzConnect:TerminalBlock_MetzConnect_360381_1x01_Horizontal_ScrewM3.0, F.Cu at (119.2, 64.9)
- added K1: SW_SPDT, footprint_switch:TE_3-1437561-8, F.Cu at (126.7, 85.7)
- added L1: L, footprint_switch:74437529203221, F.Cu at (157.2, 67.2)
- added LED_TRACO1: CQY99, LED_SMD:LED_0805_2012Metric, F.Cu at (125.4, 64.6)
- added R_TRACO1: R, Resistor_SMD:R_0805_2012Metric, F.Cu at (125.4, 60.5)
- C1, C6: footprint Capacitor_THT:CP_Radial_D13.0mm_P5.00mm -> Capacitor_SMD:C_0805_2012Metric
- C2, C4: footprint Capacitor_THT:CP_Radial_D5.0mm_P2.50mm -> Capacitor_SMD:C_0805_2012Metric
- C3, C5: footprint Capacitor_THT:C_Disc_D3.8mm_W2.6mm_P2.50mm -> Capacitor_SMD:C_0805_2012Metric
- D1, D2: footprint Package_TO_SOT_THT:TO-220-2_Vertical -> Package_TO_SOT_SMD:TO-263-2
- J1: value Screw_Terminal_01x02 -> DC IN
- J3: value Screw_Terminal_01x02 -> OUT
- LED1, LED2, LED4, LED5: footprint LED_THT:LED_D5.0mm_IRGrey -> LED_SMD:LED_0805_2012Metric
- R1, R10, R11, R12, R13, R2, R3, R4, R6, R7, R8, R9: footprint Resistor_THT:R_Axial_DIN0204_L3.6mm_D1.6mm_P7.62mm_Horizontal -> Resistor_SMD:R_0805_2012Metric
- T2, T3: value IRF4905 -> IRF4905S; footprint Package_TO_SOT_THT:TO-220-3_Vertical -> Package_TO_SOT_SMD:TO-263-2
- U1, U3: footprint Package_DIP:DIP-8_W7.62mm -> Package_DIP:SMDIP-8_W7.62mm
- U4: moved to B.Cu
- moved R9 157.7 mm to (216.1, 53.0)
- moved R10 157.7 mm to (216.0, 57.5)
- moved J3 153.9 mm to (216.9, 83.4), turned to -90 degrees
- moved R3 144.3 mm to (189.1, 90.0), turned to 90 degrees
- moved R4 142.4 mm to (186.9, 93.4), turned to -90 degrees
- moved R8 132.1 mm to (189.9, 57.2), turned to -90 degrees
- moved LED2 129.0 mm to (185.3, 90.0), turned to 90 degrees
- moved R7 128.6 mm to (186.1, 57.2), turned to -90 degrees
- moved D1 124.4 mm to (199.0, 69.6), turned to -90 degrees
- moved R1 115.0 mm to (144.3, 99.0)
- moved T2 114.6 mm to (214.5, 69.9), turned to -90 degrees
- moved C6 110.7 mm to (139.4, 104.0), turned to -90 degrees
- moved LED1 110.1 mm to (149.7, 100.8), turned to 180 degrees
- moved R2 109.3 mm to (139.6, 99.0)
- moved C5 109.3 mm to (198.1, 80.0), turned to 90 degrees
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Connections:
- C1 pad 1: Net-(D3-K) -> Net-(J1-Pin_2)
- C4 pad 2: Net-(U3-VEE) -> Net-(D1-K)
- C5 pad 2: Net-(U3-VEE) -> Net-(D1-K)
- T2 pad 2: Net-(D2-A) -> Net-(D1-A)
- T2 pad 3: Net-(D1-A) -> Net-(D2-A)
- U3 pad 5: Net-(U3-VEE) -> Net-(D1-K)
- U5 pad 1: Net-(K1-A) -> Net-(J4-Pin_2)
- U5 pad 2: Net-(D1-A) -> Net-(J4-Pin_1)
- U5 pad 4: Net-(U3-VEE) -> Net-(D1-K)
Routing:
- net Net-(D1-A): track 0.00 -> 314.2 mm, vias 0 -> 10
- net Net-(D1-K): track 0.00 -> 181.5 mm, vias 0 -> 4
- net Net-(J2-Pin_1): track 0.00 -> 178.7 mm, vias 0 -> 5
- net Net-(D2-K): track 0.00 -> 132.3 mm, vias 0 -> 4
- net Net-(K1-A): track 0.00 -> 104.6 mm
- net Net-(R9-Pad1): track 0.00 -> 101.0 mm
- net Net-(U3-VCC): track 0.00 -> 93.0 mm, vias 0 -> 2
- net Net-(D2-A): track 0.00 -> 86.0 mm, vias 0 -> 4
- net Net-(U2-A0): track 0.00 -> 62.7 mm, vias 0 -> 1
- net Net-(U2-D9): track 0.00 -> 53.4 mm, vias 0 -> 1
- net Net-(R7-Pad1): track 0.00 -> 51.0 mm, vias 0 -> 2
- net Net-(U2-A4): track 0.00 -> 44.4 mm, vias 0 -> 1
- net Net-(U2-A5): track 0.00 -> 43.0 mm, vias 0 -> 2
- net Net-(U2-3V3): track 0.00 -> 41.9 mm
- net Net-(J1-Pin_2): track 0.00 -> 33.4 mm
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Other:
- board outline added: 105.7 x 75.9 mm
