File: Buck Boost.kicad_pcb (KiCad board)
At the start: 2 copper layers, 145 x 107.2 mm, 52 parts, among them J1 Screw_Terminal_01x02, J2 Screw_Terminal_01x02, J3 Screw_Terminal_01x02, J4 Screw_Terminal_01x02, J5 Screw_Terminal_01x02, K1 SW_SPDT, K2 Jumper_2_Bridged, T2 IRF4905, T3 IRF4905, U1 HCPL-3120, U2 arduino, U3 HCPL-3120, U4 ER_OLEDM0.91_1x-I2C, U5 TMA-1512S

Commit message: V0.2
Routing:
- net Net-(J2-Pin_1): track 275.6 -> 301.6 mm
- net Net-(U2-D5): track 51.9 -> 58.4 mm
- net Net-(U2-D4): track 44.9 -> 51.4 mm
- net Net-(U2-D3): track 45.3 -> 51.8 mm
- net Net-(U2-D2): track 47.7 -> 54.2 mm
Changed lines of the file:
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@@
 			)
 		)
+		(model "${KIPRJMOD}/3Dmodels/282836-2.stp"
+			(offset
+				(xyz 2.5 -4 5)
+			)
+			(scale
+				(xyz 1 1 1)
+			)
+			(rotate
+				(xyz -90 -0 -0)
+			)
+		)
 	)
 	(footprint "Package_DIP:DIP-8_W7.62mm"
@@
 		)
 		(embedded_fonts no)
+		(model "${KIPRJMOD}/3Dmodels/RAD-DY-GF_3.stp"
+			(offset
+				(xyz 5 -3.5 30.5)
+			)
+			(scale
+				(xyz 1 1 1)
+			)
+			(rotate
+				(xyz -0 -180 -0)
+			)
+		)
 	)
 	(footprint "LED_THT:LED_D5.0mm_IRGrey"
@@
 			)
 		)
+		(model "${KIPRJMOD}/3Dmodels/282836-2.stp"
+			(offset
+				(xyz 2.5 -4 5.5)
+			)
+			(scale
+				(xyz 1 1 1)
+			)
+			(rotate
+				(xyz -90 -0 -0)
+			)
+		)
 	)
 	(footprint "Heatsink_laborator:Heasink_lab"
@@
 		)
 		(embedded_fonts no)
+		(model "${KIPRJMOD}/3Dmodels/RAD-DY-GF_3.stp"
+			(offset
+				(xyz 5 -3.5 30.5)
+			)
+			(scale
+				(xyz 1 1 1)
+			)
+			(rotate
+				(xyz -0 -180 -0)
+			)
+		)
 	)
 	(footprint "Resistor_THT:R_Axial_DIN0204_L3.6mm_D1.6mm_P7.62mm_Horizontal"
@@
 			)
 			(rotate
-				(xyz 0 0 0)
+				(xyz -0 -0 -0)
+			)
+		)
+		(model "${KIPRJMOD}/3Dmodels/282836-2.stp"
+			(offset
+				(xyz 2.5 -3.5 5.5)
+			)
+			(scale
+				(xyz 1 1 1)
+			)
+			(rotate
+				(xyz -90 -0 -0)
 			)
 		)
@@
 			)
 		)
+		(model "${KIPRJMOD}/3Dmodels/TMA 1505S--3DModel-STEP-56544.STEP"
+			(offset
+				(xyz -2.5 -7.5 1)
+			)
+			(scale
+				(xyz 1 1 1)
+			)
+			(rotate
+				(xyz -90 -0 90)
+			)
+		)
 	)
 	(footprint "Resistor_THT:R_Axial_DIN0204_L3.6mm_D1.6mm_P7.62mm_Horizontal"
@@
 		)
 		(embedded_fonts no)
+		(model "${KIPRJMOD}/3Dmodels/RAD-DY-GF_3.stp"
+			(offset
+				(xyz 5 -3.5 30.5)
+			)
+			(scale
+				(xyz 1 1 1)
+			)
+			(rotate
+				(xyz -0 -180 -0)
+			)
+		)
 	)
 	(footprint "Bobina:Bobina 470uH 3A"
@@
 		)
 		(embedded_fonts no)
+		(model "${KIPRJMOD}/3Dmodels/DPO-3.0-33.stp"
+			(offset
+				(xyz 0 -0.5 16.5)
+			)
+			(scale
+				(xyz 1.8 1.6 1.7)
+			)
+			(rotate
+				(xyz -0 -0 -0)
+			)
+		)
 	)
 	(footprint "Heatsink_laborator:Heasink_lab"
@@
 		)
 		(embedded_fonts no)
+		(model "${KIPRJMOD}/3Dmodels/RAD-DY-GF_3.stp"
+			(offset
+				(xyz 5 -3.5 30.5)
+			)
+			(scale
+				(xyz 1 1 1)
+			)
+			(rotate
+				(xyz -0 -180 -0)
+			)
+		)
 	)
 	(footprint "Package_TO_SOT_THT:TO-220-3_Vertical"
@@
 			)
 		)
+		(model "${KIPRJMOD}/3Dmodels/282836-2.stp"
+			(offset
+				(xyz 2.5 -4 6)
+			)
+			(scale
+				(xyz 1 1 1)
+			)
+			(rotate
+				(xyz -90 -0 -0)
+			)
+		)
 	)
 	(footprint "Package_TO_SOT_THT:TO-220-2_Vertical"
@@
 		)
 		(embedded_fonts no)
+		(model "${KIPRJMOD}/3Dmodels/MTS-1xx-A2-blue.step"
+			(offset
+				(xyz 0 0 0)
+			)
+			(scale
+				(xyz 1 1 1)
+			)
+			(rotate
+				(xyz -0 -0 -90)
+			)
+		)
 	)
 	(footprint "Display:ER_OLEDM0.91_1x-I2C"
@@
 			)
 		)
+		(model "${KIPRJMOD}/3Dmodels/OLED 128 x 32 Display Assembly.step"
+			(offset
+				(xyz 4 -18 4)
+			)
+			(scale
+				(xyz 1 1 1)
+			)
+			(rotate
+				(xyz -0 -0 90)
+			)
+		)
 	)
 	(footprint "Capacitor_THT:C_Disc_D3.8mm_W2.6mm_P2.50mm"
@@
 			)
 		)
+		(model "${KIPRJMOD}/3Dmodels/282836-2.stp"
+			(offset
+				(xyz 2.5 -4 5)
+			)
+			(scale
+				(xyz 1 1 1)
+			)
+			(rotate
+				(xyz -90 -0 -0)
+			)
+		)
 	)
 	(footprint "Button_Switch_THT:SW_PUSH_6mm_H5mm"
@@
 		(embedded_fonts no)
 		(model "${KICAD10_3DMODEL_DIR}/Module.3dshapes/Arduino_Nano_WithMountingHoles.step"
+			(hide yes)
 			(offset
 				(xyz 0 0 0)
 			)
 			(scale
-				(xyz 1 1 1)
+				(xyz 0 1 1)
 			)
 			(rotate
-				(xyz 0 0 0)
+				(xyz -90 -0 -0)
 			)
 		)
-		(model "C:/Program Files/KiCad/10.0/3D_Models/arduino nano.IGS"
+		(model "${KIPRJMOD}/3Dmodels/arduino nano.STEP"
 			(offset
-				(xyz 0 0 0)
+				(xyz 0 0 4)
 			)
 			(scale
@@
 			)
 			(rotate
-				(xyz 0 0 0)
+				(xyz -90 -0 90)
 			)
 		)
@@
 	)
 	(segment
+		(start 124.85 151)
+		(end 124.85 157.5)
+		(width 1.5)
+		(layer "F.Cu")
+		(net "Net-(J2-Pin_1)")
+	)
+	(segment
 		(start 77.1275 139.8325)
 		(end 76.0825 139.8325)
@@
 	)
 	(segment
+		(start 107.75 151)
+		(end 107.75 157.5)
+		(width 1.5)
+		(layer "F.Cu")
+		(net "Net-(J2-Pin_1)")
+	)
+	(segment
 		(start 78.9 136.3)
 		(end 78.9675 136.2325)
@@
 	)
 	(segment
+		(start 116.3 151)
+		(end 116.3 157.5)
+		(width 1.5)
+		(layer "F.Cu")
+		(net "Net-(J2-Pin_1)")
+	)
+	(segment
 		(start 76.35 135.95)
 		(end 77.1975 135.1025)
@@
 	)
 	(segment
+		(start 99.2 151)
+		(end 99.2 157.5)
+		(width 1.5)
+		(layer "F.Cu")
+		(net "Net-(J2-Pin_1)")
+	)
+	(segment
 		(start 106.811523 108.188477)
 		(end 106.9375 108.0625)
@@
 	)
 	(segment
+		(start 120.8 151)
+		(end 120.8 157.5)
+		(width 1.5)
+		(layer "F.Cu")
+		(net "Net-(U2-D3)")
+	)
+	(segment
 		(start 97.5175 119.2225)
 		(end 105.641 127.346)
@@
 	)
 	(segment
+		(start 129.35 151)
+		(end 129.35 157.5)
+		(width 1.5)
+		(layer "F.Cu")
+		(net "Net-(U2-D2)")
+	)
+	(segment
 		(start 100.0575 119.2225)
 		(end 106.554 125.719)
@@
 	)
 	(segment
+		(start 103.7 151)
+		(end 103.7 157.5)
+		(width 1.5)
+		(layer "F.Cu")
+		(net "Net-(U2-D5)")
+	)
+	(segment
 		(start 92.4375 119.2225)
 		(end 103.815 130.6)
@@
 	)
 	(segment
+		(start 112.25 151)
+		(end 112.25 157.5)
+		(width 1.5)
+		(layer "F.Cu")
+		(net "Net-(U2-D4)")
+	)
+	(segment

Commit message: v0.2\
Parts:
- added +Vin: TestPoint, TestPoint:TestPoint_THTPad_D3.0mm_Drill1.5mm, F.Cu at (69.5, 82.4)
- added -Vin: TestPoint, TestPoint:TestPoint_THTPad_D3.0mm_Drill1.5mm, F.Cu at (72.6, 96.7)
- added D10: TestPoint, TestPoint:TestPoint_THTPad_D3.0mm_Drill1.5mm, F.Cu at (71.0, 109.9)
- added D9: TestPoint, TestPoint:TestPoint_THTPad_D3.0mm_Drill1.5mm, F.Cu at (77.8, 109.5)
- added J5: TestPoint, TestPoint:TestPoint_THTPad_D3.0mm_Drill1.5mm, F.Cu at (173.4, 144.2)
- added J6: TestPoint, TestPoint:TestPoint_THTPad_D3.0mm_Drill1.5mm, F.Cu at (164.1, 145.0)
- renumbered C9 to C2, C2 to C3, C3 to C4, C4 to C5, C5 to C6, C6 to C7, D1 to D3, D2 to D4, Dreapta1 to Dreapta, HS4 to HS2, HS2 to HS4, J4 to J2, J2 to J3, J5 to J4, J3 to J7, Jos1 to Jos, LED7 to LED2, LED2 to LED4, LED4 to LED6, R9 to R10, R10 to R11, R6 to R12, R12 to R13, R13 to R14, R15 to R3, R5 to R4, R4 to R5, R3 to R6, R11 to R7, R7 to R8, R8 to R9, Stanga1 to Stanga, Sus1 to Sus, T3 to T1, U4 to U2, U2 to U3, U3 to U4
Routing:
- net Net-(D3-A): track 288.3 -> 296.6 mm, vias 3 -> 1
- net Net-(R10-Pad1): track 132.4 -> 128.6 mm
- net Net-(U3-D2): track 54.2 -> 57.1 mm
- net Net-(U3-D4): track 51.4 -> 54.3 mm
- net Net-(U3-D3): track 51.8 -> 54.4 mm
- net Net-(U3-D5): track 58.4 -> 60.7 mm
- net Net-(J1-Pin_2): track 38.6 -> 37.9 mm, vias 1 -> 0
- net Net-(U3-D9): track 35.4 -> 35.8 mm, vias 2 -> 1
- net Net-(U3-D10): vias 1 -> 0
- net Net-(J3-Pin_1): vias 5 -> 4
- net Net-(D4-K): vias 1 -> 0
- added copper zone on B.Cu, net (none)
- added copper zone on F.Cu, net (none)
Other:
- board text added: "Vies+"
- board text added: "Vies-"
- board text removed: "D10"
- board text removed: "Iesire"
